File: rev1.0/pcb/pcb.kicad_pcb (KiCad board)
At the start: 2 copper layers, 3.6 x 3.3 mm, 217 parts, among them J1 AVR-ISP-6, J2 USB4120-03-C, SW1 SW_Push, U1 ATMEGA32U4, U2 USBLC6-2SC6, Y1 16MHz

Commit message: pcb layout done
Parts:
- added D116: BAV70, Package_TO_SOT_SMD:SOT-23, B.Cu at (184.2, 223.3)
- added D117: BAV70, Package_TO_SOT_SMD:SOT-23, B.Cu at (169.5, 227.7)
- added D118: BAV70, Package_TO_SOT_SMD:SOT-23, B.Cu at (150.0, 214.4)
- added D119: BAV70, Package_TO_SOT_SMD:SOT-23, B.Cu at (159.7, 218.8)
- added D120: BAV70, Package_TO_SOT_SMD:SOT-23, B.Cu at (169.5, 209.9)
- added D121: SMF5.0CA, Diode_SMD:D_SOD-123F, B.Cu at (183.9, 247.9)
- added MX67: lft, 0xcb:SW_Hotswap_Kailh_1.00u, F.Cu at (357.7, 174.6)
- D1, D10, D11, D12, D13, D14, D2, D3, D4, D5, D6, D7, D8, D9: value SK6812MINI-E -> WS2812B; footprint 0xcb:MX_SK6812MINI-E -> LED_SMD:LED_WS2812B_PLCC4_5.0x5.0mm_P3.2mm; moved to B.Cu
- D115: value SMF5.0CA -> BAV70; footprint Diode_SMD:D_SOD-123F -> Package_TO_SOT_SMD:SOT-23
- D69, D70, D71, D72, D73, D74, D75, D76, D77, D78: value WS2812B -> SK6812MINI-E; footprint LED_SMD:LED_WS2812B_PLCC4_5.0x5.0mm_P3.2mm -> 0xcb:MX_SK6812MINI-E; moved to F.Cu
- D79, D80, D81, D82, D83: value BAV70 -> SK6812MINI-E; footprint Package_TO_SOT_SMD:SOT-23 -> 0xcb:MX_SK6812MINI-E; moved to F.Cu
- MX58: footprint 0xcb:SW_Hotswap_Kailh_1.25u -> 0xcb:SW_Hotswap_Kailh_1.00u
- MX61: footprint 0xcb:SW_Hotswap_Kailh_6.25u -> 0xcb:SW_Hotswap_Kailh_1.25u
- MX62: footprint 0xcb:SW_Hotswap_Kailh_1.25u -> 0xcb:SW_Hotswap_Kailh_6.25u
- MX64: value lft -> MX; footprint 0xcb:SW_Hotswap_Kailh_1.00u -> 0xcb:SW_Hotswap_Kailh_1.25u
- MX65: value dwn -> lft
- MX66: value lft -> dwn
- moved D29 585.3 mm to (357.7, 98.4)
- moved D23 547.7 mm to (224.4, 98.4)
- moved D38 526.2 mm to (233.9, 117.4)
- moved D44 523.3 mm to (357.7, 117.4)
- moved D40 519.2 mm to (272.0, 117.4)
- moved D55 509.0 mm to (276.8, 136.5)
- moved D42 492.6 mm to (310.1, 117.4)
- moved D28 492.2 mm to (329.1, 98.4)
- moved D19 487.6 mm to (148.2, 98.4)
- moved D22 483.0 mm to (205.3, 98.4)
- moved D36 482.6 mm to (195.8, 117.4)
- moved D49 473.6 mm to (162.5, 136.5)
- moved D57 472.9 mm to (326.8, 136.5)
- moved D25 466.4 mm to (262.5, 98.4)
- moved D48 465.2 mm to (143.4, 136.5)
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Connections:
- D1 pad 4: /RGB -> Net-(D1-Pad4)
- D101 pad 2: unconnected-(D101-Pad2) -> Net-(D101-Pad2)
- D102 pad 1: unconnected-(D102-Pad1) -> Net-(D102-Pad1)
- D103 pad 1: unconnected-(D103-Pad1) -> Net-(D103-Pad1)
- D103 pad 3: R3 -> R2
- D104 pad 3: R3 -> R2
- D105 pad 3: R3 -> R2
- D106 pad 2: Net-(D106-Pad2) -> unconnected-(D106-Pad2)
- D106 pad 3: R3 -> R2
- D107 pad 1: Net-(D107-Pad1) -> unconnected-(D107-Pad1)
- D107 pad 3: R3 -> R2
- D108 pad 1: Net-(D108-Pad1) -> unconnected-(D108-Pad1)
- D11 pad 2: Net-(D11-Pad2) -> Net-(D10-Pad4)
- D11 pad 4: Net-(D10-Pad2) -> Net-(D11-Pad4)
- D110 pad 3: R4 -> R3
- D111 pad 3: R4 -> R3
- D112 pad 3: R4 -> R3
- D113 pad 3: R4 -> R3
- D114 pad 1: unconnected-(D114-Pad1) -> Net-(D114-Pad1)
- D114 pad 3: R4 -> R3
- D115 pad 1: GND -> unconnected-(D115-Pad1)
- D115 pad 2: Net-(C15-Pad1) -> Net-(D115-Pad2)
- D12 pad 2: Net-(D12-Pad2) -> Net-(D11-Pad4)
- D12 pad 4: Net-(D11-Pad2) -> Net-(D12-Pad4)
- D13 pad 2: Net-(D13-Pad2) -> Net-(D12-Pad4)
- D13 pad 4: Net-(D12-Pad2) -> Net-(D13-Pad4)
- D14 pad 2: Net-(D14-Pad2) -> Net-(D13-Pad4)
- D14 pad 4: Net-(D13-Pad2) -> /RGB
- D15 pad 4: Net-(D14-Pad2) -> Net-(D1-Pad2)
- D16 pad 4: Net-(D16-Pad4) -> Net-(D15-Pad2)
- D17 pad 2: Net-(D16-Pad4) -> Net-(D17-Pad2)
- D17 pad 4: Net-(D17-Pad4) -> Net-(D16-Pad2)
- D18 pad 2: Net-(D17-Pad4) -> Net-(D18-Pad2)
- D18 pad 4: Net-(D18-Pad4) -> Net-(D17-Pad2)
- D19 pad 2: Net-(D18-Pad4) -> Net-(D19-Pad2)
- D19 pad 4: Net-(D19-Pad4) -> Net-(D18-Pad2)
- D2 pad 2: Net-(D2-Pad2) -> Net-(D1-Pad4)
- D2 pad 4: Net-(D1-Pad2) -> Net-(D2-Pad4)
- D20 pad 2: Net-(D19-Pad4) -> Net-(D20-Pad2)
- D20 pad 4: Net-(D20-Pad4) -> Net-(D19-Pad2)
- D21 pad 2: Net-(D20-Pad4) -> Net-(D21-Pad2)
- D21 pad 4: Net-(D21-Pad4) -> Net-(D20-Pad2)
- D22 pad 2: Net-(D21-Pad4) -> Net-(D22-Pad2)
- D22 pad 4: Net-(D22-Pad4) -> Net-(D21-Pad2)
- D23 pad 2: Net-(D22-Pad4) -> Net-(D23-Pad2)
- D23 pad 4: Net-(D23-Pad4) -> Net-(D22-Pad2)
- D24 pad 2: Net-(D23-Pad4) -> Net-(D24-Pad2)
- D24 pad 4: Net-(D24-Pad4) -> Net-(D23-Pad2)
- D25 pad 2: Net-(D24-Pad4) -> Net-(D25-Pad2)
- D25 pad 4: Net-(D25-Pad4) -> Net-(D24-Pad2)
- D26 pad 2: Net-(D25-Pad4) -> Net-(D26-Pad2)
- D26 pad 4: Net-(D26-Pad4) -> Net-(D25-Pad2)
- D27 pad 2: Net-(D26-Pad4) -> Net-(D27-Pad2)
- D27 pad 4: Net-(D27-Pad4) -> Net-(D26-Pad2)
- D28 pad 2: Net-(D27-Pad4) -> Net-(D28-Pad2)
- D28 pad 4: Net-(D28-Pad4) -> Net-(D27-Pad2)
- D29 pad 2: Net-(D28-Pad4) -> Net-(D29-Pad2)
- D29 pad 4: Net-(D29-Pad4) -> Net-(D28-Pad2)
- D3 pad 2: Net-(D3-Pad2) -> Net-(D2-Pad4)
- D3 pad 4: Net-(D2-Pad2) -> Net-(D3-Pad4)
- D30 pad 2: Net-(D29-Pad4) -> Net-(D30-Pad2)
- D30 pad 4: Net-(D15-Pad2) -> Net-(D30-Pad4)
- D31 pad 2: Net-(D31-Pad2) -> Net-(D30-Pad4)
- D31 pad 4: Net-(D16-Pad2) -> Net-(D31-Pad4)
- D32 pad 2: Net-(D32-Pad2) -> Net-(D31-Pad4)
- D32 pad 4: Net-(D31-Pad2) -> Net-(D32-Pad4)
- D33 pad 2: Net-(D33-Pad2) -> Net-(D32-Pad4)
- D33 pad 4: Net-(D32-Pad2) -> Net-(D33-Pad4)
- D34 pad 2: Net-(D34-Pad2) -> Net-(D33-Pad4)
- D34 pad 4: Net-(D33-Pad2) -> Net-(D34-Pad4)
- D35 pad 2: Net-(D35-Pad2) -> Net-(D34-Pad4)
- D35 pad 4: Net-(D34-Pad2) -> Net-(D35-Pad4)
- D36 pad 2: Net-(D36-Pad2) -> Net-(D35-Pad4)
- D36 pad 4: Net-(D35-Pad2) -> Net-(D36-Pad4)
- D37 pad 2: Net-(D37-Pad2) -> Net-(D36-Pad4)
- D37 pad 4: Net-(D36-Pad2) -> Net-(D37-Pad4)
- D38 pad 2: Net-(D38-Pad2) -> Net-(D37-Pad4)
- D38 pad 4: Net-(D37-Pad2) -> Net-(D38-Pad4)
- D39 pad 2: Net-(D39-Pad2) -> Net-(D38-Pad4)
- D39 pad 4: Net-(D38-Pad2) -> Net-(D39-Pad4)
- D4 pad 2: Net-(D4-Pad2) -> Net-(D3-Pad4)
- D4 pad 4: Net-(D3-Pad2) -> Net-(D4-Pad4)
- D40 pad 2: Net-(D40-Pad2) -> Net-(D39-Pad4)
- D40 pad 4: Net-(D39-Pad2) -> Net-(D40-Pad4)
- D41 pad 2: Net-(D41-Pad2) -> Net-(D40-Pad4)
- D41 pad 4: Net-(D40-Pad2) -> Net-(D41-Pad4)
- D42 pad 2: Net-(D42-Pad2) -> Net-(D41-Pad4)
- D42 pad 4: Net-(D41-Pad2) -> Net-(D42-Pad4)
- D43 pad 2: Net-(D43-Pad2) -> Net-(D42-Pad4)
- D43 pad 4: Net-(D42-Pad2) -> Net-(D43-Pad4)
- D44 pad 2: Net-(D44-Pad2) -> Net-(D43-Pad4)
- D44 pad 4: Net-(D43-Pad2) -> Net-(D29-Pad2)
- D45 pad 4: Net-(D45-Pad4) -> Net-(D30-Pad2)
- D46 pad 2: Net-(D45-Pad4) -> Net-(D46-Pad2)
- D46 pad 4: Net-(D46-Pad4) -> Net-(D45-Pad2)
- D47 pad 2: Net-(D46-Pad4) -> Net-(D47-Pad2)
- D47 pad 4: Net-(D47-Pad4) -> Net-(D46-Pad2)
- D48 pad 2: Net-(D47-Pad4) -> Net-(D48-Pad2)
- D48 pad 4: Net-(D48-Pad4) -> Net-(D47-Pad2)
- D49 pad 2: Net-(D48-Pad4) -> Net-(D49-Pad2)
- D49 pad 4: Net-(D49-Pad4) -> Net-(D48-Pad2)
- D5 pad 2: Net-(D5-Pad2) -> Net-(D4-Pad4)
- D5 pad 4: Net-(D4-Pad2) -> Net-(D5-Pad4)
- D50 pad 2: Net-(D49-Pad4) -> Net-(D50-Pad2)
- D50 pad 4: Net-(D50-Pad4) -> Net-(D49-Pad2)
- D51 pad 2: Net-(D50-Pad4) -> Net-(D51-Pad2)
- D51 pad 4: Net-(D51-Pad4) -> Net-(D50-Pad2)
- D52 pad 2: Net-(D51-Pad4) -> Net-(D52-Pad2)
- D52 pad 4: Net-(D52-Pad4) -> Net-(D51-Pad2)
- D53 pad 2: Net-(D52-Pad4) -> Net-(D53-Pad2)
- D53 pad 4: Net-(D53-Pad4) -> Net-(D52-Pad2)
- D54 pad 2: Net-(D53-Pad4) -> Net-(D54-Pad2)
- D54 pad 4: Net-(D54-Pad4) -> Net-(D53-Pad2)
- D55 pad 2: Net-(D54-Pad4) -> Net-(D55-Pad2)
- D55 pad 4: Net-(D55-Pad4) -> Net-(D54-Pad2)
- D56 pad 2: Net-(D55-Pad4) -> Net-(D56-Pad2)
- D56 pad 4: Net-(D56-Pad4) -> Net-(D55-Pad2)
- D57 pad 2: Net-(D56-Pad4) -> Net-(D57-Pad2)
- D57 pad 4: Net-(D57-Pad4) -> Net-(D56-Pad2)
- D58 pad 2: Net-(D57-Pad4) -> Net-(D58-Pad2)
- D58 pad 4: Net-(D44-Pad2) -> Net-(D57-Pad2)
- D59 pad 4: Net-(D45-Pad2) -> Net-(D59-Pad4)
- D6 pad 2: Net-(D6-Pad2) -> Net-(D5-Pad4)
- D6 pad 4: Net-(D5-Pad2) -> Net-(D6-Pad4)
- D60 pad 2: Net-(D60-Pad2) -> Net-(D59-Pad4)
- D60 pad 4: Net-(D59-Pad2) -> Net-(D60-Pad4)
- D61 pad 2: Net-(D61-Pad2) -> Net-(D60-Pad4)
- D61 pad 4: Net-(D60-Pad2) -> Net-(D61-Pad4)
- D62 pad 2: Net-(D62-Pad2) -> Net-(D61-Pad4)
- D62 pad 4: Net-(D61-Pad2) -> Net-(D62-Pad4)
- D63 pad 2: Net-(D63-Pad2) -> Net-(D62-Pad4)
- D63 pad 4: Net-(D62-Pad2) -> Net-(D63-Pad4)
- D64 pad 2: Net-(D64-Pad2) -> Net-(D63-Pad4)
- D64 pad 4: Net-(D63-Pad2) -> Net-(D64-Pad4)
- D65 pad 2: Net-(D65-Pad2) -> Net-(D64-Pad4)
- D65 pad 4: Net-(D64-Pad2) -> Net-(D65-Pad4)
- D66 pad 2: Net-(D66-Pad2) -> Net-(D65-Pad4)
- D66 pad 4: Net-(D65-Pad2) -> Net-(D66-Pad4)
- D67 pad 2: Net-(D67-Pad2) -> Net-(D66-Pad4)
- D67 pad 4: Net-(D66-Pad2) -> Net-(D67-Pad4)
- D68 pad 2: Net-(D68-Pad2) -> Net-(D67-Pad4)
- D68 pad 4: Net-(D67-Pad2) -> Net-(D68-Pad4)
- D69 pad 2: unconnected-(D69-Pad2) -> Net-(D68-Pad4)
- D7 pad 2: Net-(D7-Pad2) -> Net-(D6-Pad4)
- D7 pad 4: Net-(D6-Pad2) -> Net-(D7-Pad4)
- D72 pad 4: Net-(D72-Pad4) -> Net-(D58-Pad2)
- D73 pad 2: Net-(D72-Pad4) -> Net-(D73-Pad2)
- D73 pad 4: Net-(D73-Pad4) -> Net-(D59-Pad2)
- D74 pad 2: Net-(D73-Pad4) -> Net-(D74-Pad2)
- D74 pad 4: Net-(D74-Pad4) -> Net-(D73-Pad2)
- D75 pad 2: Net-(D74-Pad4) -> Net-(D75-Pad2)
- D75 pad 4: Net-(D75-Pad4) -> Net-(D74-Pad2)
- D76 pad 2: Net-(D75-Pad4) -> Net-(D76-Pad2)
- D76 pad 4: Net-(D76-Pad4) -> Net-(D75-Pad2)
- D77 pad 2: Net-(D76-Pad4) -> Net-(D77-Pad2)
- D77 pad 4: Net-(D77-Pad4) -> Net-(D76-Pad2)
- D78 pad 2: Net-(D77-Pad4) -> Net-(D78-Pad2)
- D78 pad 4: Net-(D68-Pad2) -> Net-(D77-Pad2)
- D79 pad 1: Net-(D79-Pad1) -> VCC
- D79 pad 3: R0 -> GND
- D8 pad 2: Net-(D8-Pad2) -> Net-(D7-Pad4)
- D8 pad 4: Net-(D7-Pad2) -> Net-(D8-Pad4)
- D80 pad 1: Net-(D80-Pad1) -> VCC
- D80 pad 3: R0 -> GND
- D81 pad 1: Net-(D81-Pad1) -> VCC
- D81 pad 3: R0 -> GND
- D82 pad 1: Net-(D82-Pad1) -> VCC
- D82 pad 3: R0 -> GND
- D83 pad 1: Net-(D83-Pad1) -> VCC
- D83 pad 2: Net-(D83-Pad2) -> unconnected-(D83-Pad2)
- D83 pad 3: R0 -> GND
- D86 pad 1: unconnected-(D86-Pad1) -> Net-(D86-Pad1)
- D87 pad 3: R1 -> R0
- D88 pad 3: R1 -> R0
- D89 pad 3: R1 -> R0
- D9 pad 2: Net-(D10-Pad4) -> Net-(D8-Pad4)
- D9 pad 4: Net-(D8-Pad2) -> Net-(D10-Pad2)
- D90 pad 3: R1 -> R0
- D91 pad 1: Net-(D91-Pad1) -> unconnected-(D91-Pad1)
- D91 pad 3: R1 -> R0
- D94 pad 1: unconnected-(D94-Pad1) -> Net-(D94-Pad1)
- D95 pad 3: R2 -> R1
- D96 pad 3: R2 -> R1
- D97 pad 3: R2 -> R1
- D98 pad 3: R2 -> R1
- D99 pad 1: Net-(D99-Pad1) -> unconnected-(D99-Pad1)
- D99 pad 3: R2 -> R1
- MX1 pad 2: Net-(D79-Pad2) -> Net-(D84-Pad2)
- MX10 pad 2: Net-(D83-Pad1) -> Net-(D88-Pad1)
- MX11 pad 2: Net-(D84-Pad2) -> Net-(D89-Pad2)
- MX12 pad 2: Net-(D84-Pad1) -> Net-(D89-Pad1)
- MX13 pad 2: Net-(D85-Pad2) -> Net-(D90-Pad2)
- MX14 pad 2: Net-(D85-Pad1) -> Net-(D90-Pad1)
- MX15 pad 2: Net-(D86-Pad2) -> Net-(D91-Pad2)
- MX16 pad 2: Net-(D87-Pad2) -> Net-(D92-Pad2)
- MX17 pad 2: Net-(D87-Pad1) -> Net-(D92-Pad1)
- MX18 pad 2: Net-(D88-Pad2) -> Net-(D93-Pad2)
- MX19 pad 2: Net-(D88-Pad1) -> Net-(D93-Pad1)
- MX2 pad 2: Net-(D79-Pad1) -> Net-(D84-Pad1)
- MX20 pad 2: Net-(D89-Pad2) -> Net-(D94-Pad2)
- MX21 pad 2: Net-(D89-Pad1) -> Net-(D94-Pad1)
- MX22 pad 2: Net-(D90-Pad2) -> Net-(D95-Pad2)
- MX23 pad 2: Net-(D90-Pad1) -> Net-(D95-Pad1)
- MX24 pad 2: Net-(D91-Pad2) -> Net-(D96-Pad2)
- MX25 pad 2: Net-(D91-Pad1) -> Net-(D96-Pad1)
- MX26 pad 2: Net-(D92-Pad2) -> Net-(D97-Pad2)
- MX27 pad 2: Net-(D92-Pad1) -> Net-(D97-Pad1)
- MX28 pad 2: Net-(D93-Pad2) -> Net-(D98-Pad2)
- MX29 pad 2: Net-(D93-Pad1) -> Net-(D98-Pad1)
- MX3 pad 2: Net-(D80-Pad2) -> Net-(D85-Pad2)
- MX30 pad 2: Net-(D94-Pad2) -> Net-(D99-Pad2)
- MX31 pad 2: Net-(D95-Pad2) -> Net-(D100-Pad2)
- MX32 pad 2: Net-(D95-Pad1) -> Net-(D100-Pad1)
- MX33 pad 2: Net-(D96-Pad2) -> Net-(D101-Pad2)
- MX34 pad 2: Net-(D96-Pad1) -> Net-(D101-Pad1)
- MX35 pad 2: Net-(D97-Pad2) -> Net-(D102-Pad2)
- MX36 pad 2: Net-(D97-Pad1) -> Net-(D102-Pad1)
- MX37 pad 2: Net-(D98-Pad2) -> Net-(D103-Pad2)
- MX38 pad 2: Net-(D98-Pad1) -> Net-(D103-Pad1)
- MX39 pad 2: Net-(D99-Pad2) -> Net-(D104-Pad2)
- MX4 pad 2: Net-(D80-Pad1) -> Net-(D85-Pad1)
- MX40 pad 2: Net-(D99-Pad1) -> Net-(D104-Pad1)
- MX41 pad 2: Net-(D100-Pad2) -> Net-(D105-Pad2)
- MX42 pad 2: Net-(D100-Pad1) -> Net-(D105-Pad1)
- MX43 pad 2: Net-(D101-Pad1) -> Net-(D106-Pad1)
- MX44 pad 2: Net-(D102-Pad2) -> Net-(D107-Pad2)
- MX45 pad 2: Net-(D103-Pad2) -> Net-(D108-Pad2)
- MX46 pad 2: Net-(D104-Pad2) -> Net-(D109-Pad2)
- MX47 pad 2: Net-(D104-Pad1) -> Net-(D109-Pad1)
- MX48 pad 2: Net-(D105-Pad2) -> Net-(D110-Pad2)
- MX49 pad 2: Net-(D105-Pad1) -> Net-(D110-Pad1)
- MX5 pad 2: Net-(D81-Pad2) -> Net-(D86-Pad2)
- MX50 pad 2: Net-(D106-Pad2) -> Net-(D111-Pad2)
- MX51 pad 2: Net-(D106-Pad1) -> Net-(D111-Pad1)
- MX52 pad 2: Net-(D107-Pad2) -> Net-(D112-Pad2)
- MX53 pad 2: Net-(D107-Pad1) -> Net-(D112-Pad1)
- MX54 pad 2: Net-(D108-Pad2) -> Net-(D113-Pad2)
- MX55 pad 2: Net-(D108-Pad1) -> Net-(D113-Pad1)
- MX56 pad 2: Net-(D109-Pad2) -> Net-(D114-Pad2)
- MX57 pad 2: Net-(D109-Pad1) -> Net-(D114-Pad1)
- MX58 pad 1: C0 -> C13
- MX58 pad 2: Net-(D110-Pad2) -> Net-(D115-Pad2)
- MX59 pad 1: C1 -> C0
- MX59 pad 2: Net-(D110-Pad1) -> Net-(D116-Pad2)
- MX6 pad 2: Net-(D81-Pad1) -> Net-(D86-Pad1)
- MX60 pad 1: C2 -> C1
- MX60 pad 2: Net-(D111-Pad2) -> Net-(D116-Pad1)
- MX61 pad 1: C7 -> C2
- MX61 pad 2: Net-(D111-Pad1) -> Net-(D117-Pad2)
- MX62 pad 1: C10 -> C7
- MX62 pad 2: Net-(D112-Pad2) -> Net-(D117-Pad1)
- MX63 pad 1: C11 -> C10
- MX63 pad 2: Net-(D112-Pad1) -> Net-(D118-Pad2)
- MX64 pad 1: C12 -> C11
- MX64 pad 2: Net-(D113-Pad2) -> Net-(D118-Pad1)
- MX65 pad 1: C13 -> C12
- MX65 pad 2: Net-(D113-Pad1) -> Net-(D119-Pad2)
- MX66 pad 2: Net-(D114-Pad2) -> Net-(D119-Pad1)
- MX7 pad 2: Net-(D82-Pad2) -> Net-(D87-Pad2)
- MX8 pad 2: Net-(D82-Pad1) -> Net-(D87-Pad1)
- MX9 pad 2: Net-(D83-Pad2) -> Net-(D88-Pad2)
Routing:
- added copper zone on B.Cu, net GND
- added copper zone on F.Cu, net GND
Other:
- board size 3.6 x 3.3 mm -> 305.5 x 96 mm

Commit message: Columns and Rows
Parts:
- moved D99 221.0 mm to (348.2, 107.9), turned to 90 degrees
- moved D91 220.4 mm to (348.2, 92.4), turned to 90 degrees
- moved D115 202.6 mm to (348.2, 149.5), turned to 90 degrees
- moved D106 201.5 mm to (343.4, 127.0), turned to 90 degrees
- moved D107 201.4 mm to (348.2, 127.0), turned to 90 degrees
- moved D90 197.4 mm to (310.1, 92.4), turned to 90 degrees
- moved D120 183.4 mm to (348.2, 168.6), turned to 90 degrees
- moved D114 182.7 mm to (329.1, 146.0), turned to 90 degrees
- moved D119 176.7 mm to (329.1, 168.6), turned to 90 degrees
- moved D98 174.0 mm to (319.6, 111.4), turned to 90 degrees
- moved D105 157.8 mm to (286.3, 130.5), turned to 90 degrees
- moved D89 150.3 mm to (272.0, 92.4), turned to 90 degrees
- moved D84 149.8 mm to (81.5, 92.4), turned to 90 degrees
- moved D97 148.6 mm to (281.5, 111.4), turned to 90 degrees
- moved D88 143.8 mm to (233.9, 92.4), turned to 90 degrees
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Routing:
- net R4: track 0.00 -> 271.1 mm
- net R0: track 0.00 -> 269.3 mm
- net R1: track 0.00 -> 265.2 mm
- net R3: track 0.00 -> 264.0 mm
- net R2: track 0.00 -> 261.7 mm
- net C7: track 0.00 -> 99.2 mm, vias 0 -> 5
- net C2: track 0.00 -> 93.7 mm, vias 0 -> 5
- net C10: track 0.00 -> 93.2 mm, vias 0 -> 5
- net C11: track 0.00 -> 93.2 mm, vias 0 -> 5
- net C12: track 0.00 -> 91.1 mm, vias 0 -> 4
- net C0: track 0.00 -> 91.0 mm, vias 0 -> 5
- net C1: track 0.00 -> 89.1 mm, vias 0 -> 4
- net C8: track 0.00 -> 71.7 mm, vias 0 -> 4
- net C4: track 0.00 -> 71.6 mm, vias 0 -> 4
- net C5: track 0.00 -> 71.6 mm, vias 0 -> 4
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
Commit message: edited schematic and fixed constraints
Parts:
- removed D121: SMF5.0CA, Diode_SMD:D_SOD-123F
- D120: value BAV70 -> SMF5.0CA; footprint Package_TO_SOT_SMD:SOT-23 -> Diode_SMD:D_SOD-123F
- J2: footprint 0xcb:MOLEX_2130830005 -> 0xcb:GCT_USB4105_REVA
- moved D99 188.9 mm to (170.3, 44.4), turned to 180 degrees
- moved D115 186.0 mm to (194.8, 44.4), turned to 180 degrees
- moved D119 180.0 mm to (194.8, 48.8), turned to 180 degrees
- moved D114 177.9 mm to (180.1, 48.8), turned to 180 degrees
- moved F1 174.1 mm to (198.8, 74.7)
- moved R3 174.1 mm to (194.6, 74.5)
- moved D106 172.3 mm to (189.9, 48.8), turned to 180 degrees
- moved D120 172.2 mm to (203.7, 74.9), turned to 180 degrees
- moved FB2 171.2 mm to (191.3, 77.0)
- moved R5 168.5 mm to (195.3, 77.4)
- moved C1 166.8 mm to (241.1, 82.8)
- moved C10 166.8 mm to (250.4, 63.2)
- moved C11 166.8 mm to (254.4, 63.2)
- moved C12 166.8 mm to (250.4, 65.8)
- moved C13 166.8 mm to (246.4, 63.2)
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Connections:
- D106 pad 1: Net-(D106-Pad1) -> unconnected-(D106-Pad1)
- D106 pad 2: unconnected-(D106-Pad2) -> Net-(D106-Pad2)
- D107 pad 3: R2 -> R3
- D108 pad 1: unconnected-(D108-Pad1) -> Net-(D108-Pad1)
- D114 pad 2: Net-(D114-Pad2) -> unconnected-(D114-Pad2)
- D115 pad 1: unconnected-(D115-Pad1) -> Net-(D115-Pad1)
- D115 pad 3: R3 -> R4
- D119 pad 2: Net-(D119-Pad2) -> unconnected-(D119-Pad2)
- D120 pad 1: unconnected-(D120-Pad1) -> GND
- D120 pad 2: Net-(D120-Pad2) -> Net-(C15-Pad1)
- D91 pad 1: unconnected-(D91-Pad1) -> Net-(D91-Pad1)
- D91 pad 2: Net-(D91-Pad2) -> unconnected-(D91-Pad2)
- D99 pad 1: unconnected-(D99-Pad1) -> Net-(D99-Pad1)
- D99 pad 2: Net-(D99-Pad2) -> unconnected-(D99-Pad2)
- MX15 pad 1: C13 -> C14
- MX15 pad 2: Net-(D91-Pad2) -> Net-(D91-Pad1)
- MX30 pad 1: C13 -> C14
- MX30 pad 2: Net-(D99-Pad2) -> Net-(D99-Pad1)
- MX43 pad 2: Net-(D106-Pad1) -> Net-(D106-Pad2)
- MX44 pad 1: C13 -> C14
- MX44 pad 2: Net-(D107-Pad2) -> unconnected-(MX44-Pad2)
- MX45 pad 2: Net-(D108-Pad2) -> Net-(D107-Pad2)
- MX46 pad 2: Net-(D109-Pad2) -> Net-(D108-Pad2)
- MX47 pad 2: Net-(D109-Pad1) -> Net-(D108-Pad1)
- MX48 pad 2: Net-(D110-Pad2) -> Net-(D109-Pad2)
- MX49 pad 2: Net-(D110-Pad1) -> Net-(D109-Pad1)
- MX50 pad 2: Net-(D111-Pad2) -> Net-(D110-Pad2)
- MX51 pad 2: Net-(D111-Pad1) -> Net-(D110-Pad1)
- MX52 pad 2: Net-(D112-Pad2) -> Net-(D111-Pad2)
- MX53 pad 2: Net-(D112-Pad1) -> Net-(D111-Pad1)
- MX54 pad 2: Net-(D113-Pad2) -> Net-(D112-Pad2)
- MX55 pad 2: Net-(D113-Pad1) -> Net-(D112-Pad1)
- MX56 pad 2: Net-(D114-Pad2) -> Net-(D113-Pad2)
- MX57 pad 2: Net-(D114-Pad1) -> Net-(D113-Pad1)
- MX58 pad 1: C13 -> C14
- MX58 pad 2: Net-(D115-Pad2) -> Net-(D114-Pad1)
- MX59 pad 2: Net-(D116-Pad2) -> Net-(D115-Pad2)
- MX60 pad 2: Net-(D116-Pad1) -> Net-(D115-Pad1)
- MX61 pad 2: Net-(D117-Pad2) -> Net-(D116-Pad2)
- MX62 pad 2: Net-(D117-Pad1) -> Net-(D116-Pad1)
- MX63 pad 2: Net-(D118-Pad2) -> Net-(D117-Pad2)
- MX64 pad 2: Net-(D118-Pad1) -> Net-(D117-Pad1)
- MX65 pad 2: Net-(D119-Pad2) -> Net-(D118-Pad2)
- MX66 pad 2: Net-(D119-Pad1) -> Net-(D118-Pad1)
- MX67 pad 1: C13 -> C14
- MX67 pad 2: Net-(D120-Pad2) -> Net-(D119-Pad1)
- U1 pad 8: C13 -> C14
Routing:
- net R4: track 271.1 -> 0.00 mm
- net R0: track 269.3 -> 0.00 mm
- net R1: track 265.2 -> 0.00 mm
- net R3: track 264.0 -> 0.00 mm
- net R2: track 261.7 -> 0.00 mm
- net C7: track 99.2 -> 0.00 mm, vias 5 -> 0
- net C2: track 93.7 -> 0.00 mm, vias 5 -> 0
- net C10: track 93.2 -> 0.00 mm, vias 5 -> 0
- net C11: track 93.2 -> 0.00 mm, vias 5 -> 0
- net C12: track 91.1 -> 0.00 mm, vias 4 -> 0
- net C0: track 91.0 -> 0.00 mm, vias 5 -> 0
- net C1: track 89.1 -> 0.00 mm, vias 4 -> 0
- net C8: track 71.7 -> 0.00 mm, vias 4 -> 0
- net C4: track 71.6 -> 0.00 mm, vias 4 -> 0
- net C5: track 71.6 -> 0.00 mm, vias 4 -> 0
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
Commit message: Did the rows... again
Parts:
- moved D114 195.9 mm to (348.2, 149.5), turned to 90 degrees
- moved D119 194.6 mm to (348.2, 168.6), turned to 90 degrees
- moved D99 188.9 mm to (348.2, 107.9), turned to 90 degrees
- moved D118 181.8 mm to (329.1, 168.6), turned to 90 degrees
- moved D106 178.1 mm to (348.2, 130.5), turned to 90 degrees
- moved D113 171.4 mm to (329.1, 146.0), turned to 90 degrees
- moved D115 166.5 mm to (83.9, 168.6), turned to 90 degrees
- moved D91 163.1 mm to (348.2, 92.4), turned to 90 degrees
- moved D117 145.5 mm to (274.4, 168.6), turned to 90 degrees
- moved D90 135.7 mm to (310.1, 92.4), turned to 90 degrees
- moved D107 135.3 mm to (88.6, 146.0), turned to 90 degrees
- moved D116 131.7 mm to (131.5, 168.6), turned to 90 degrees
- moved D105 130.1 mm to (286.3, 130.5), turned to 90 degrees
- moved D98 128.9 mm to (319.6, 111.4), turned to 90 degrees
- moved D84 126.0 mm to (81.5, 92.4), turned to 90 degrees
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Connections:
- D106 pad 1: unconnected-(D106-Pad1) -> Net-(D106-Pad1)
- MX44 pad 1: C14 -> unconnected-(MX44-Pad1)
- MX44 pad 2: unconnected-(MX44-Pad2) -> Net-(D106-Pad1)
Routing:
- net R4: track 0.00 -> 276.1 mm
- net R0: track 0.00 -> 275.8 mm
- net R1: track 0.00 -> 270.2 mm
- net R3: track 0.00 -> 267.7 mm
- net R2: track 0.00 -> 264.8 mm
- net Net-(D116-Pad1): track 0.00 -> 68.6 mm
- net Net-(D90-Pad1): track 0.00 -> 25.8 mm
- net Net-(D100-Pad1): track 0.00 -> 23.4 mm
- net Net-(D92-Pad1): track 0.00 -> 22.7 mm
- net Net-(D115-Pad1): track 0.00 -> 21.0 mm
- net Net-(D98-Pad1): track 0.00 -> 21.0 mm
- net Net-(D117-Pad1): track 0.00 -> 21.0 mm
- net Net-(D88-Pad2): track 0.00 -> 20.2 mm
- net Net-(D91-Pad1): track 0.00 -> 16.2 mm
- net Net-(D106-Pad1): track 0.00 -> 16.2 mm
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