File: rev1.0/pcb/pcb.kicad_pcb (KiCad board)
At the start: 2 copper layers, 305.5 x 96 mm, 223 parts, among them J1 AVR-ISP-6, J2 USB4120-03-C, SW1 SW_Push, U1 ATMEGA32U4, U2 USBLC6-2SC6, Y1 16MHz

Commit message: RGB LED Stuff
Parts:
- moved C13 213.2 mm to (67.8, 179.7), turned to -90 degrees
- moved C11 198.0 mm to (72.6, 141.6), turned to -90 degrees
- moved C12 197.3 mm to (77.3, 160.7), turned to -90 degrees
- moved C9 191.7 mm to (66.5, 103.5), turned to -90 degrees
- moved C10 189.7 mm to (70.2, 122.5), turned to -90 degrees
- moved SW1 129.0 mm to (174.5, 178.1), turned to -90 degrees
- moved J1 121.3 mm to (180.7, 178.5), turned to -90 degrees
- moved U1 97.7 mm to (214.7, 173.3), turned to 45 degrees
Connections:
- MX44 pad 1: unconnected-(MX44-Pad1) -> C14
Routing:
- net VCC: track 0.00 -> 1377.5 mm
- net C13: track 0.00 -> 95.4 mm, vias 0 -> 5
- net C7: track 0.00 -> 95.2 mm, vias 0 -> 5
- net C2: track 0.00 -> 94.2 mm, vias 0 -> 5
- net C10: track 0.00 -> 93.8 mm, vias 0 -> 5
- net C11: track 0.00 -> 93.8 mm, vias 0 -> 5
- net C0: track 0.00 -> 92.8 mm, vias 0 -> 5
- net C12: track 0.00 -> 91.4 mm, vias 0 -> 4
- net C1: track 0.00 -> 91.2 mm, vias 0 -> 4
- net C14: track 0.00 -> 85.6 mm, vias 0 -> 5
- net C5: track 0.00 -> 72.0 mm, vias 0 -> 4
- net C3: track 0.00 -> 71.9 mm, vias 0 -> 4
- net C6: track 0.00 -> 71.9 mm, vias 0 -> 4
- net C4: track 0.00 -> 71.9 mm, vias 0 -> 4
- net Net-(D80-Pad2): track 0.00 -> 67.6 mm
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