File: rev1.0/pcb/RGB.kicad_sch (KiCad schematic)
At the start: 84 parts

Commit message: pcb layout done
Parts:
- removed D78: WS2812B, LED_SMD:LED_WS2812B_PLCC4_5.0x5.0mm_P3.2mm, symbol LED:WS2812B
- added D10, D11, D12, D13, D14: WS2812B, LED_SMD:LED_WS2812B_PLCC4_5.0x5.0mm_P3.2mm, symbol LED:WS2812B
- added D79: SK6812MINI-E, 0xcb:MX_SK6812MINI-E, symbol 0xcb:SK6812MINI-E
- renumbered D69 to D1, D1 to D15, D2 to D16, D3 to D17, D4 to D18, D5 to D19, D70 to D2, D6 to D20, D7 to D21, D8 to D22, D9 to D23, D10 to D24, D11 to D25, D12 to D26, D13 to D27, D14 to D28, D15 to D29, D71 to D3, D16 to D30, D17 to D31, D18 to D32, D19 to D33, D20 to D34, D21 to D35, D22 to D36, D23 to D37, D24 to D38, D25 to D39, D72 to D4, D26 to D40, D27 to D41, D28 to D42, D29 to D43, D30 to D44, D31 to D45, D32 to D46, D33 to D47, D34 to D48, D35 to D49, D73 to D5, D36 to D50, D37 to D51, D38 to D52, D39 to D53, D40 to D54, D41 to D55, D42 to D56, D43 to D57, D44 to D58, D45 to D59, D74 to D6, D46 to D60, D47 to D61, D48 to D62, D49 to D63, D50 to D64, D51 to D65, D52 to D66, D53 to D67, D54 to D68, D55 to D69, D75 to D7, D56 to D70, D57 to D71, D58 to D72, D59 to D73, D60 to D74, D61 to D75, D62 to D76, D63 to D77, D64 to D78, D76 to D8, D65 to D80, D66 to D81, D67 to D82, D68 to D83, D77 to D9
Connections:
- net GND: now also D10.3 (VSS), D11.3 (VSS), D12.3 (VSS), D13.3 (VSS), D14.3 (VSS), D79.3 (VSS)
- net RGB: now also D14.4 (DIN); no longer D15.4 (DIN)
- net VCC: now also D10.1 (VDD), D11.1 (VDD), D12.1 (VDD), D13.1 (VDD), D14.1 (VDD), D79.1 (VDD)
- net at D80.4 (DIN): now also D79.2 (DOUT); no longer D78.2 (DOUT)
- net at D1.2 (DOUT): now also D15.4 (DIN)
- net at D9.4 (DIN): now also D10.2 (DOUT)
- new net: D11.4 (DIN), D12.2 (DOUT)
- new net: D12.4 (DIN), D13.2 (DOUT)
- new net: D13.4 (DIN), D14.2 (DOUT)
- new net: D10.4 (DIN), D11.2 (DOUT)
- new net: D78.2 (DOUT), D79.4 (DIN)
Other:
- moved on the sheet: C10, C11, C12, C13, C14, C9, D1, D15, D16, D17, D18, D19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

Commit message: addes HS LEDs
Parts:
- removed D1, D10, D11, D12, D13, D14, D2, D3, D4, D5, D6, D7, D8, D9: WS2812B, LED_SMD:LED_WS2812B_PLCC4_5.0x5.0mm_P3.2mm, symbol LED:WS2812B
- added D1, D10, D11, D12, D13, D14, D2, D3, D4, D5, D6, D7, D8, D9: SK6812MINI-HS, 0xcb:SK6812MINI-HS, symbol 0xcb:SK6812MINI-HS
Connections:
- net GND: now also D1.1 (VSS), D10.1 (VSS), D11.1 (VSS), D12.1 (VSS), D13.1 (VSS), D14.1 (VSS), D2.1 (VSS), D3.1 (VSS), D4.1 (VSS), D5.1 (VSS), D6.1 (VSS), D7.1 (VSS), D8.1 (VSS), D9.1 (VSS)
- net RGB: now also D15.4 (DIN)
- net VCC: now also D1.3 (VDD), D10.3 (VDD), D11.3 (VDD), D12.3 (VDD), D13.3 (VDD), D14.3 (VDD), D2.3 (VDD), D3.3 (VDD), D4.3 (VDD), D5.3 (VDD), D6.3 (VDD), D7.3 (VDD), D8.3 (VDD), D9.3 (VDD)
- net at D16.2 (DOUT): now also D2.2 (DIN); no longer D17.4 (DIN)
- net at D16.4 (DIN): now also D1.4 (DOUT); no longer D15.2 (DOUT)
- net at D24.2 (DOUT): now also D10.2 (DIN); no longer D25.4 (DIN)
- net at D24.4 (DIN): now also D9.4 (DOUT); no longer D23.2 (DOUT)
- net at D23.4 (DIN): now also D8.4 (DOUT); no longer D22.2 (DOUT)
- net at D22.4 (DIN): now also D7.4 (DOUT); no longer D21.2 (DOUT)
- net at D18.2 (DOUT): now also D4.2 (DIN); no longer D19.4 (DIN)
- net at D18.4 (DIN): now also D3.4 (DOUT); no longer D17.2 (DOUT)
- net at D19.2 (DOUT): now also D5.2 (DIN); no longer D20.4 (DIN)
- net at D25.2 (DOUT): now also D11.2 (DIN); no longer D26.4 (DIN)
- net at D26.2 (DOUT): now also D12.2 (DIN); no longer D27.4 (DIN)
- net at D28.2 (DOUT): now also D14.2 (DIN); no longer D29.4 (DIN)
- net at D28.4 (DIN): now also D13.4 (DOUT); no longer D27.2 (DOUT)
- net at D20.2 (DOUT): now also D6.2 (DIN); no longer D21.4 (DIN)
- new net: D17.4 (DIN), D2.4 (DOUT)
- new net: D23.2 (DOUT), D9.2 (DIN)
- new net: D22.2 (DOUT), D8.2 (DIN)
- new net: D19.4 (DIN), D4.4 (DOUT)
- new net: D10.4 (DOUT), D25.4 (DIN)
- new net: D12.4 (DOUT), D27.4 (DIN)
- new net: D17.2 (DOUT), D3.2 (DIN)
- new net: D11.4 (DOUT), D26.4 (DIN)
- new net: D21.4 (DIN), D6.4 (DOUT)
- new net: D14.4 (DOUT), D29.4 (DIN)
- new net: D13.2 (DIN), D27.2 (DOUT)
- new net: D21.2 (DOUT), D7.2 (DIN)
- new net: D1.2 (DIN), D15.2 (DOUT)
- new net: D20.4 (DIN), D5.4 (DOUT)
Other:
- moved on the sheet: C10, C11, C12, C13, C14, C9, D15, D16, D17, D18, D19, D20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
