File: rev1.0/pcb/RGB.kicad_sch (KiCad schematic)
At the start: 89 parts

Commit message: rp2040 port: updated schematic and fixed footprints
Parts:
- C10, C11, C12, C13, C14, C9: footprint Capacitor_SMD:C_0603_1608Metric -> Capacitor_SMD:C_0201_0603Metric
Other:
- moved on the sheet: C10, C11, C12, C13, C14, C9, D1, D10, D11, D12, D13, D14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

Commit message: fixup and add prod
Parts:
- C10, C11, C12, C13, C14, C9: LCSC (none) -> C576431
- D1, D10, D11, D12, D13, D14, D2, D3, D4, D5, D6, D7, D8, D9: LCSC (none) -> C2922787
- D15, D16, D17, D18, D19, D20, D21, D22, D23, D24, D25, D26, D27, D28, D29, D30, D31, D32, D33, D34, D35, D36, D37, D38, D39, D40, D41, D42, D43, D44, D45, D46, D47, D48, D49, D50, D51, D52, D53, D54, D55, D56, D57, D58, D59, D60, D61, D62, D63, D64, D65, D66, D67, D68, D69, D70, D71, D72, D73, D74, D75, D76, D77, D78, D79, D80, D81, D82, D83: LCSC (none) -> C5149201
