File: rev1.0/pcb/matrix.kicad_sch (KiCad schematic)
At the start: 102 parts

Commit message: pcb layout done
Parts:
- added D115: BAV70, Package_TO_SOT_SMD:SOT-23, symbol 0xcb:BAV70
- added MX58: MX, 0xcb:SW_Hotswap_Kailh_1.00u, symbol 0xcb:MX
- renumbered D95 to D100, D96 to D101, D97 to D102, D98 to D103, D99 to D104, D100 to D105, D101 to D106, D102 to D107, D103 to D108, D104 to D109, D105 to D110, D106 to D111, D107 to D112, D108 to D113, D109 to D114, D110 to D116, D111 to D117, D112 to D118, D113 to D119, D114 to D120, D79 to D84, D80 to D85, D81 to D86, D82 to D87, D83 to D88, D84 to D89, D85 to D90, D86 to D91, D87 to D92, D88 to D93, D89 to D94, D90 to D95, D91 to D96, D92 to D97, D93 to D98, D94 to D99, MX58 to MX59, MX59 to MX60, MX60 to MX61, MX61 to MX62, MX62 to MX63, MX63 to MX64, MX64 to MX65, MX65 to MX66, MX66 to MX67
Connections:
- net C14: now also MX58.1 (COL)
- net R3: now also D115.3 (K)
- new net: D115.2 (A2), MX58.2 (ROW)
- no-connect marks 6 -> 7

Commit message: edited schematic and fixed constraints
Parts:
- removed D106: BAV70, Package_TO_SOT_SMD:SOT-23, symbol 0xcb:BAV70
- renumbered D107 to D106, D108 to D107, D109 to D108, D110 to D109, D111 to D110, D112 to D111, D113 to D112, D114 to D113, D115 to D114, D116 to D115, D117 to D116, D118 to D117, D119 to D118, D120 to D119
Connections:
- net at MX30.2 (ROW): now also D99.1 (A1); no longer D99.2 (A2)
- net at D114.1 (A1): now also MX58.2 (ROW)
- net at D114.2 (A2): no longer MX58.2 (ROW)
- net at MX67.2 (ROW): now also D119.1 (A1); no longer D119.2 (A2)
- net at MX43.2 (ROW): now also D106.2 (A2)
- net at MX44.2 (ROW): no longer D106.2 (A2)
- net at MX15.2 (ROW): now also D91.1 (A1); no longer D91.2 (A2)
- no-connect marks 7 -> 5
Other:
- moved on the sheet: D106

Commit message: Did the rows... again
Connections:
- net C14: no longer MX44.1 (COL)
- net at MX44.2 (ROW): now also D106.1 (A1)
Changed lines of the file:
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@@
   (junction (at 176.276 58.547) (diameter 0) (color 0 0 0 0))
   (junction (at 176.276 69.85) (diameter 0) (color 0 0 0 0))
+  (junction (at 183.388 58.547) (diameter 0) (color 0 0 0 0))
   (junction (at 186.436 35.9664) (diameter 0) (color 0 0 0 0))
   (junction (at 186.436 47.2694) (diameter 0) (color 0 0 0 0))
@@
     (pin "2")
   )
-  (symbol (lib_id "0xcb:MX") (at 179.578 58.5724 0) (unit 1)
-    (in_bom yes) (on_board yes)
-    (property "Reference" "MX44" (id 0) (at 178.6255 56.4134 0))
-    (property "Value" "MX" (id 1) (at 179.2605 59.4614 0)
-      (effects (font (size 0.508 0.508)))
-    )
-    (property "Footprint" "0xcb:SW_Hotswap_Kailh_1.00u" (id 2) (at 180.848 56.0324 0)
-      (effects (font (size 1.27 1.27)) hide)
-    )
-    (property "Datasheet" "" (id 3) (at 180.848 56.0324 0)
-      (effects (font (size 1.27 1.27)) hide)
-    )
+  (symbol (lib_id "0xcb:MX") (at 179.578 58.547 0) (unit 1)
+    (in_bom yes) (on_board yes)
+    (property "Reference" "MX44" (id 0) (at 178.6255 56.388 0))
+    (property "Value" "MX" (id 1) (at 179.2605 59.436 0)
+      (effects (font (size 0.508 0.508)))
+    )
+    (property "Footprint" "0xcb:SW_Hotswap_Kailh_1.00u" (id 2) (at 180.848 56.007 0)
+      (effects (font (size 1.27 1.27)) hide)
+    )
+    (property "Datasheet" "" (id 3) (at 180.848 56.007 0)
+      (effects (font (size 1.27 1.27)) hide)
+    )

Commit message: RGB LED Stuff
Connections:
- net C14: now also MX44.1 (COL)
Changed lines of the file:
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@@
   (junction (at 176.276 58.547) (diameter 0) (color 0 0 0 0))
   (junction (at 176.276 69.85) (diameter 0) (color 0 0 0 0))
-  (junction (at 183.388 58.547) (diameter 0) (color 0 0 0 0))
   (junction (at 186.436 35.9664) (diameter 0) (color 0 0 0 0))
   (junction (at 186.436 47.2694) (diameter 0) (color 0 0 0 0))
+  (junction (at 186.436 58.547) (diameter 0) (color 0 0 0 0))
   (junction (at 186.436 58.5709) (diameter 0) (color 0 0 0 0))
   (junction (at 186.436 69.8794) (diameter 0) (color 0 0 0 0))
@@
     (stroke (width 0) (type default) (color 0 0 0 0))
   )
-  (wire (pts (xy 183.388 58.5709) (xy 183.388 58.5724))
-    (stroke (width 0) (type default) (color 0 0 0 0))
-  )
   (wire (pts (xy 183.388 88.7984) (xy 163.068 88.7984))
     (stroke (width 0) (type default) (color 0 0 0 0))
@@
     (stroke (width 0) (type solid) (color 0 0 0 0))
   )
-  (wire (pts (xy 186.436 47.2694) (xy 186.436 58.5709))
-    (stroke (width 0) (type default) (color 0 0 0 0))
-  )
-  (wire (pts (xy 186.436 58.5709) (xy 183.388 58.5709))
-    (stroke (width 0) (type default) (color 0 0 0 0))
-  )
+  (wire (pts (xy 186.436 47.2694) (xy 186.436 58.547))
+    (stroke (width 0) (type default) (color 0 0 0 0))
+  )
+  (wire (pts (xy 186.436 58.547) (xy 183.388 58.547))
+    (stroke (width 0) (type default) (color 0 0 0 0))
+  )
+  (wire (pts (xy 186.436 58.547) (xy 186.436 58.5709))
+    (stroke (width 0) (type default) (color 0 0 0 0))
+  )
