File: rev1.0/pcb/usb.kicad_sch (KiCad schematic)
At the start: 12 parts, among them J2 USB4120-03-C, U2 USBLC6-2SC6

Commit message: pcb layout done
Parts:
- renumbered D115 to D121
Changed lines of the file:
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@@
   (symbol (lib_id "power:VCC") (at 108.966 51.689 0) (unit 1)
     (in_bom yes) (on_board yes)
-    (property "Reference" "#PWR023" (id 0) (at 108.966 55.499 0)
+    (property "Reference" "#PWR021" (id 0) (at 108.966 55.499 0)
       (effects (font (size 1.27 1.27)) hide)
     )
@@
   (symbol (lib_id "power:VCC") (at 124.968 35.433 0) (unit 1)
     (in_bom yes) (on_board yes)
-    (property "Reference" "#PWR021" (id 0) (at 124.968 39.243 0)
+    (property "Reference" "#PWR019" (id 0) (at 124.968 39.243 0)
       (effects (font (size 1.27 1.27)) hide)
     )
@@
   (symbol (lib_id "power:GND") (at 70.358 95.631 0) (unit 1)
     (in_bom yes) (on_board yes)
-    (property "Reference" "#PWR026" (id 0) (at 70.358 101.981 0)
+    (property "Reference" "#PWR024" (id 0) (at 70.358 101.981 0)
       (effects (font (size 1.27 1.27)) hide)
     )
@@
   (symbol (lib_id "power:GND") (at 100.838 43.053 0) (unit 1)
     (in_bom yes) (on_board yes)
-    (property "Reference" "#PWR022" (id 0) (at 100.838 49.403 0)
+    (property "Reference" "#PWR020" (id 0) (at 100.838 49.403 0)
       (effects (font (size 1.27 1.27)) hide)
     )
@@
   (symbol (lib_id "power:GND") (at 100.838 55.499 0) (unit 1)
     (in_bom yes) (on_board yes)
-    (property "Reference" "#PWR024" (id 0) (at 100.838 61.849 0)
+    (property "Reference" "#PWR022" (id 0) (at 100.838 61.849 0)
       (effects (font (size 1.27 1.27)) hide)
     )
@@
   (symbol (lib_id "power:GND") (at 108.966 75.819 0) (unit 1)
     (in_bom yes) (on_board yes)
-    (property "Reference" "#PWR025" (id 0) (at 108.966 82.169 0)
+    (property "Reference" "#PWR023" (id 0) (at 108.966 82.169 0)
       (effects (font (size 1.27 1.27)) hide)
     )
@@
   (symbol (lib_id "Device:D_TVS") (at 100.838 39.243 90) (unit 1)
     (in_bom yes) (on_board yes)
-    (property "Reference" "D115" (id 0) (at 102.362 36.7029 90)
+    (property "Reference" "D121" (id 0) (at 102.362 36.7029 90)
       (effects (font (size 1.27 1.27)) (justify right))
     )

Commit message: edited schematic and fixed constraints
Parts:
- J2: footprint 0xcb:MOLEX_2130830005 -> 0xcb:GCT_USB4105_REVA
- renumbered D121 to D120
Changed lines of the file:
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@@
   (symbol (lib_id "Device:D_TVS") (at 100.838 39.243 90) (unit 1)
     (in_bom yes) (on_board yes)
-    (property "Reference" "D121" (id 0) (at 102.362 36.7029 90)
+    (property "Reference" "D120" (id 0) (at 102.362 36.7029 90)
       (effects (font (size 1.27 1.27)) (justify right))
     )
@@
     (property "Reference" "J2" (id 0) (at 77.597 41.021 0))
     (property "Value" "USB4120-03-C" (id 1) (at 77.851 43.561 0))
-    (property "Footprint" "0xcb:MOLEX_2130830005" (id 2) (at 81.788 63.119 0)
+    (property "Footprint" "0xcb:GCT_USB4105_REVA" (id 2) (at 81.788 63.119 0)
       (effects (font (size 1.27 1.27)) hide)
     )
